File: PCB - KiCad/DSKY_driver_clr/DSKY_driver.sch (KiCad schematic (older format))
At the start: 229 parts, among them IC3 ATSAMD21E, J1 FX6-60S, J2 FX6-60S, J3 FX6-60S, J4 CUI_power_jack, Q2 reset, U1 HV507, U2 LT3468, U3 AP2204K-3.3, U4 AP2204K-5.0, U5 HV507, U6 LT3468, U7 HV507, U8 CD40109B, X1 USB_micro

Commit message: Fine tuning resistor placement
Parts:
- C10: value 10n -> 10nF
- C15, C16, C17: value .22u -> .22uF
- C5, C9: value 6.3uF -> 6.8uF
- C7, C8: value 2.2u -> 2.2uF
- J4: value CUI_power_jack -> PJ-006B-SMT
- R10, R100, R101, R102, R103, R104, R105, R106, R107, R108, R109, R11, R110, R111, R112, R113, R114, R115, R116, R117, R118, R119, R12, R120, R121, R122, R123, R124, R125, R126, R127, R128, R129, R13, R130, R131, R132, R133, R134, R135, R136, R137, R138, R139, R14, R140, R141, R142, R143, R144, R145, R146, R147, R148, R149, R15, R150, R151, R152, R153, R154, R155, R156, R157, R158, R159, R16, R160, R161, R162, R163, R164, R165, R166, R167, R168, R169, R17, R170, R171, R172, R173, R174, R175, R176, R177, R178, R179, R18, R180, R181, R182, R183, R184, R19, R20, R21, R22, R23, R24, R25, R26, R27, R28, R29, R30, R31, R32, R33, R34, R35, R36, R37, R38, R39, R40, R41, R42, R43, R44, R45, R46, R47, R48, R49, R5, R50, R51, R52, R53, R54, R55, R56, R57, R58, R59, R6, R60, R61, R62, R63, R64, R65, R66, R67, R68, R69, R7, R70, R71, R72, R73, R74, R75, R76, R77, R78, R79, R8, R80, R81, R82, R83, R84, R85, R86, R87, R88, R89, R9, R90, R91, R92, R93, R94, R95, R96, R97, R98, R99: value 100K -> 75K
- X1: value USB_micro -> Molex 105133
